Commit message: Basic gazebo sim(unsolved weights and accleration errors)

File: description/corrected_robot_core.xacro (robot description, xacro)
@@ -46,5 +46,5 @@
     </link>
     <gazebo reference="chassis">
-	<material>Gazebo/white</material>
+	    <material>Gazebo/White</material>
     </gazebo>
     <!-- LEFT WHEEL LINK -->
@@ -72,5 +72,5 @@
     </link>
     <gazebo reference="left_wheel">
-	<material>Gazebo/blue</material>
+	    <material>Gazebo/Blue</material>
     </gazebo>
     <!-- RIGHT WHEEL LINK -->
@@ -98,5 +98,5 @@
     </link>
     <gazebo reference="right_wheel">
-	<material>Gazebo/blue</material>
+	    <material>Gazebo/Blue</material>
     </gazebo>
     <!-- CASTER WHEEL LINKS -->
@@ -124,7 +124,7 @@
     </link>
     <gazebo reference="caster_wheel_fl">
-	<material>Gazebo/black</material>
-    <mu1 value="0.001"></mu1>
-    <mu2 value="0.001"></mu2>
+	    <material>Gazebo/Black</material>
+        <mu1 value="0.001"></mu1>
+        <mu2 value="0.001"></mu2>
     </gazebo>
  <!-- caster_wheel_joint_fr LINK -->
@@ -151,7 +151,7 @@
     </link>
     <gazebo reference="caster_wheel_fr">
-	<material>Gazebo/black</material>
-    <mu1 value="0.001"></mu1>
-    <mu2 value="0.001"></mu2>
+	    <material>Gazebo/Black</material>
+        <mu1 value="0.001"></mu1>
+        <mu2 value="0.001"></mu2>
     </gazebo>
  <!-- caster_wheel_joint_bl LINK -->
@@ -178,7 +178,7 @@
     </link>
     <gazebo reference="caster_wheel_bl">
-	<material>Gazebo/black</material>
-    <mu1 value="0.001"></mu1>
-    <mu2 value="0.001"></mu2>
+	    <material>Gazebo/Black</material>
+        <mu1 value="0.001"></mu1>
+        <mu2 value="0.001"></mu2>
     </gazebo>
  <!-- caster_wheel_joint_br LINK -->
@@ -205,7 +205,7 @@
     </link>
     <gazebo reference="caster_wheel_br">
-	<material>Gazebo/black</material>
-    <mu1 value="0.001"></mu1>
-    <mu2 value="0.001"></mu2>
+	    <material>Gazebo/Black</material>
+        <mu1 value="0.001"></mu1>
+        <mu2 value="0.001"></mu2>
     </gazebo>
 </robot>

File: description/robot.urdf.xacro (robot description, xacro)
@@ -3,4 +3,4 @@
     <xacro:include filename="corrected_robot_core.xacro"/>
     <!-- <xacro:include filename="lidar.xacro"/>  -->
-    <!-- <xacro:include filename="gazebo_control(1).xarco"/> -->
+    <xacro:include filename="gazebo_control(1).xarco"/>
 </robot>

Commit message: Basic Gazebo Sim working(all errors fixed)

File: description/corrected_robot_core.xacro (robot description, xacro)
@@ -25,9 +25,9 @@
         <parent link="base_link" />
         <child link="chassis" />
-        <origin xyz="-0.5 0 -0.025" />
+        <origin xyz="0 0 -0.025" />
     </joint>
     <link name="chassis">
         <visual>
-            <origin xyz="0.5 0 0.1" />
+            <origin xyz="0 0 0.1" />
             <geometry>
                 <box size="1 0.7 0.2" />
@@ -105,19 +105,19 @@
         <parent link="chassis" />
         <child link="caster_wheel_fl" />
-        <origin xyz="0.9 0.3 -0.025" />
+        <origin xyz="0.4 0.2 -0.005" />
     </joint>
     <link name="caster_wheel_fl">
         <visual>
             <geometry>
-                <sphere radius="0.04"/>
-            </geometry>
-            <material name="black" />
-        </visual>
-	<collision>
-            <geometry>
-                <sphere radius="0.04"/>
-            </geometry>
-        </collision>
-	 <xacro:inertial_sphere mass="1" radius="0.04">
+                <sphere radius="0.05"/>
+            </geometry>
+            <material name="black" />
+        </visual>
+	<collision>
+            <geometry>
+                <sphere radius="0.05"/>
+            </geometry>
+        </collision>
+	 <xacro:inertial_sphere mass="1" radius="0.05">
             <origin xyz="0 0 0" rpy="0 0 0" />
         </xacro:inertial_sphere>
@@ -132,19 +132,19 @@
         <parent link="chassis" />
         <child link="caster_wheel_fr" />
-        <origin xyz="0.9 -0.3 -0.025" />
+        <origin xyz="0.4 -0.2 -0.005" />
     </joint>
     <link name="caster_wheel_fr">
         <visual>
             <geometry>
-                <sphere radius="0.04"/>
-            </geometry>
-            <material name="black" />
-        </visual>
-	<collision>
-            <geometry>
-                <sphere radius="0.04"/>
-            </geometry>
-        </collision>
-	<xacro:inertial_sphere mass="1" radius="0.04">
+                <sphere radius="0.05"/>
+            </geometry>
+            <material name="black" />
+        </visual>
+	<collision>
+            <geometry>
+                <sphere radius="0.05"/>
+            </geometry>
+        </collision>
+	<xacro:inertial_sphere mass="1" radius="0.05">
             <origin xyz="0 0 0" rpy="0 0 0" />
         </xacro:inertial_sphere>
@@ -159,19 +159,19 @@
         <parent link="chassis" />
         <child link="caster_wheel_bl" />
-        <origin xyz="0.1 0.3 -0.025" />
+        <origin xyz="-0.4 0.2 -0.005" />
     </joint>
     <link name="caster_wheel_bl">
         <visual>
             <geometry>
-                <sphere radius="0.04"/>
-            </geometry>
-            <material name="black" />
-        </visual>
-	<collision>
-            <geometry>
-                <sphere radius="0.04"/>
-            </geometry>
-        </collision>
-`	<xacro:inertial_sphere mass="1" radius="0.04">
+                <sphere radius="0.05"/>
+            </geometry>
+            <material name="black" />
+        </visual>
+	<collision>
+            <geometry>
+                <sphere radius="0.05"/>
+            </geometry>
+        </collision>
+`	<xacro:inertial_sphere mass="1" radius="0.05">
             <origin xyz="0 0 0" rpy="0 0 0" />
         </xacro:inertial_sphere>
@@ -186,19 +186,19 @@
         <parent link="chassis" />
         <child link="caster_wheel_br" />
-        <origin xyz="0.1 -0.3 -0.025" />
+        <origin xyz="-0.4 -0.2 -0.005" />
     </joint>
     <link name="caster_wheel_br">
         <visual>
             <geometry>
-                <sphere radius="0.04"/>
-            </geometry>
-            <material name="black" />
-        </visual>
-	<collision>
-            <geometry>
-                <sphere radius="0.04"/>
-            </geometry>
-        </collision>
-	<xacro:inertial_sphere mass="1" radius="0.04">
+                <sphere radius="0.05"/>
+            </geometry>
+            <material name="black" />
+        </visual>
+	<collision>
+            <geometry>
+                <sphere radius="0.05"/>
+            </geometry>
+        </collision>
+	<xacro:inertial_sphere mass="1" radius="0.05">
             <origin xyz="0 0 0" rpy="0 0 0" />
         </xacro:inertial_sphere>

Commit message: gazebo sim  working with lidar

File: description/corrected_robot_core.xacro (robot description, xacro)
@@ -36,5 +36,5 @@
         </visual>
         <collision>
-            <origin xyz="0.5 0 0.1" />
+            <origin xyz="0 0 0.1" />
             <geometry>
                 <box size="1 0.7 0.2" />

File: description/lidar.xacro (robot description, xacro)
@@ -4,5 +4,5 @@
         <parent link="chassis" />
         <child link="laser_front" />
-        <origin xyz="1.04 0.4 0.14" rpy="0 0 -${pi/4}" />
+        <origin xyz="0.5 0.35 0.14" rpy="0 0 ${pi/6}" />
     </joint>
     <link name="laser_front">
@@ -15,9 +15,91 @@
         </visual>
         <collision>
-            <origin xyz="1.03 1.03 0.14" />
+            <origin xyz="0 0 0"/>
             <geometry>
                 <box size="0.07 0.05 0.1" />
             </geometry>
         </collision>
+        <xacro:inertial_box mass="2" x="0.007" y="0.05" z="0.1">
+            <origin xyz="0 0 0" rpy="0 0 ${pi/6}" />
+        </xacro:inertial_box>
      </link>
+     <gazebo reference="laser_front">
+        <material>Gazebo/Red</material>
+        <sensor name="laser1" type="ray">
+            <pose> 0 0 0 0 0 0 </pose>
+            <visualize>true</visualize>
+            <update_rate>10</update_rate>
+            <ray>
+                <scan>
+                    <horizontal>
+                        <samples>270</samples>
+                        <min_angle>-2.35</min_angle>
+                        <max_angle>2.35</max_angle>
+                    </horizontal>
+                </scan>
+                <range>
+                    <min>0.5</min>
+                    <max>10</max>
+                </range>
+            </ray>
+            <plugin name="laser_controller_fornt" filename="libgazebo_ros_ray_sensor.so">
+                <ros>
+                    <argument>~/out:=scan_front</argument>
+                </ros>
+                <output_type>sensor_msgs/LaserScan</output_type>
+                <frame_name>laser_front</frame_name>
+            </plugin>
+        </sensor>
+    </gazebo>
+     <joint name="laser_back_joint" type="fixed">
+        <parent link="chassis" />
+        <child link="laser_back" />
+        <origin xyz="-0.5 -0.35 0.14" rpy="0 0 3.66" />
+    </joint>
+    <link name="laser_back">
+        <visual>
+            <origin xyz="0 0 0" />
+            <geometry>
+                <box size="0.07 0.05 0.1" />
+            </geometry>
+            <material name="red" />
+        </visual>
+        <collision>
+            <origin xyz="0 0 0"/>
+            <geometry>
+                <box size="0.07 0.05 0.1" />
+            </geometry>
+        </collision>
+        <xacro:inertial_box mass="2" x="0.007" y="0.05" z="0.1">
+            <origin xyz="0 0 0" rpy="0 0 3.66" />
+        </xacro:inertial_box>
+     </link>
+      <gazebo reference="laser_back">
+        <material>Gazebo/Red</material>
+        <sensor name="laser2" type="ray">
+            <pose> 0 0 0 0 0 0 </pose>
+            <visualize>true</visualize>
+            <update_rate>10</update_rate>
+            <ray>
+                <scan>
+                    <horizontal>
+                        <samples>270</samples>
+                        <min_angle>-2.35</min_angle>
+                        <max_angle>2.35</max_angle>
+                    </horizontal>
+                </scan>
+                <range>
+                    <min>0.5</min>
+                    <max>10</max>
+                </range>
+            </ray>
+            <plugin name="laser_controller_back" filename="libgazebo_ros_ray_sensor.so">
+                <ros>
+                    <argument>~/out:=scan_back</argument>
+                </ros>
+                <output_type>sensor_msgs/LaserScan</output_type>
+                <frame_name>laser_back</frame_name>
+            </plugin>
+        </sensor>
+    </gazebo>
 </robot>

File: description/robot.urdf.xacro (robot description, xacro)
@@ -2,5 +2,5 @@
 <robot xmlns:xacro="http://www.ros.org/wiki/xacro" name="robot">
     <xacro:include filename="corrected_robot_core.xacro"/>
-    <!-- <xacro:include filename="lidar.xacro"/>  -->
+    <xacro:include filename="lidar.xacro"/>
     <xacro:include filename="gazebo_control(1).xarco"/>
 </robot>
